File: HW/TestBoards/IF1_BPF_EvalBoard/IF1_BPF_EvalBoard.kicad_pcb (KiCad board)
At the start: 2 copper layers, 40 x 50 mm, 8 parts, among them J1 SMA, J2 SMA, J3 SMA, J4 SMA

Commit message: LO1 Eval Board
Parts:
- added H1: M2.5, MountingHole:MountingHole_2.7mm_M2.5_Pad, F.Cu at (125.0, 95.0)
- added H2: M2.5, MountingHole:MountingHole_2.7mm_M2.5_Pad, F.Cu at (125.0, 135.0)
- added H3: M2.5, MountingHole:MountingHole_2.7mm_M2.5_Pad, F.Cu at (155.0, 95.0)
- added H4: M2.5, MountingHole:MountingHole_2.7mm_M2.5_Pad, F.Cu at (155.0, 135.0)
- moved FL3 3.00 mm to (134.9, 124.0)
- moved FL4 3.00 mm to (144.5, 125.3)
- moved J3 3.00 mm to (120.6, 125.0)
- moved J4 3.00 mm to (159.4, 125.0)
- moved FL1 2.17 mm to (134.9, 103.7)
- moved FL2 2.17 mm to (144.8, 104.7)
- moved J1 2.17 mm to (120.6, 104.7)
- moved J2 2.17 mm to (159.5, 104.7)
Routing:
- net GND: vias 325 -> 318
