File: HW/TestBoards/IF1_BPF_EvalBoard/IF1_BPF_EvalBoard_RO4003C_60mils.kicad_pcb (KiCad board)
At the start: 2 copper layers, 40 x 30 mm, 8 parts, among them J1 SMA, J2 SMA, J3 SMA, J4 SMA

Commit message: EvalBoards in RO4003C 60 mils
Parts:
- added REF**: Grapa_0.8mm_11.9mm, GGS_Miscellaneous:Grapa_0.8mm_11.9mm, F.Cu at (122.0, 114.6)
- added REF**: Grapa_0.8mm_11.9mm, GGS_Miscellaneous:Grapa_0.8mm_11.9mm, F.Cu at (146.1, 114.6)
Changed lines of the file:
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@@
     (grid_origin 120 140)
     (pcbplotparams
-      (layerselection 0x00010fc_ffffffff)
+      (layerselection 0x0001000_ffffffff)
       (disableapertmacros false)
       (usegerberextensions false)
@@
       (outputformat 1)
       (mirror false)
-      (drillshape 1)
+      (drillshape 0)
       (scaleselection 1)
-      (outputdirectory "")
+      (outputdirectory "E:/PCBprint/Board1/IF1/")
     )
   )
@@
   (net 6 "/HPF_out2")
   (net 7 "/RF_Out2")
+  (footprint "GGS_Miscellaneous:Grapa_0.8mm_11.9mm" (layer "F.Cu")
+    (at 122.05 114.591351)
+    (attr smd)
+    (fp_text reference "REF**" (at 0 -0.5 unlocked) (layer "F.SilkS")
+      (effects (font (size 1 1) (thickness 0.15)))
+    )
+    (fp_text value "Grapa_0.8mm_11.9mm" (at 0 1 unlocked) (layer "F.Fab")
+      (effects (font (size 1 1) (thickness 0.15)))
+    )
+    (fp_text user "${REFERENCE}" (at 0 2.5 unlocked) (layer "F.Fab")
+      (effects (font (size 1 1) (thickness 0.15)))
+    )
+    (pad "" np_thru_hole circle (at 0 -3) (size 0.8 0.8) (drill 0.8) (layers F&B.Cu *.Mask))
+    (pad "" np_thru_hole circle (at 11.9 -3.032701) (size 0.8 0.8) (drill 0.8) (layers F&B.Cu *.Mask))
+  )
   (footprint "GGS_RF:JC0603C-1" (layer "F.Cu")
     (at 144.55301 132.315999)
@@
     )
   )
+  (footprint "GGS_Miscellaneous:Grapa_0.8mm_11.9mm" (layer "F.Cu")
+    (at 146.05 114.591351)
+    (attr smd)
+    (fp_text reference "REF**" (at 0 -0.5 unlocked) (layer "F.SilkS")
+      (effects (font (size 1 1) (thickness 0.15)))
+    )
+    (fp_text value "Grapa_0.8mm_11.9mm" (at 0 1 unlocked) (layer "F.Fab")
+      (effects (font (size 1 1) (thickness 0.15)))
+    )
+    (fp_text user "${REFERENCE}" (at 0 2.5 unlocked) (layer "F.Fab")
+      (effects (font (size 1 1) (thickness 0.15)))
+    )
+    (pad "" np_thru_hole circle (at 0 -3) (size 0.8 0.8) (drill 0.8) (layers F&B.Cu *.Mask))
+    (pad "" np_thru_hole circle (at 11.9 -3.032701) (size 0.8 0.8) (drill 0.8) (layers F&B.Cu *.Mask))
+  )
   (footprint "GGS_Connectors:LINX_CONSMA020.062-G" (layer "F.Cu")
     (at 159.4525 132 90)
@@
     (pts (xy 120 140) (xy 160 140))
     (height 10)
-    (gr_text "40,0000 mm" (at 140 148.85) (layer "Cmts.User")
+    (gr_text "1574,8031 mils" (at 140 148.85) (layer "Cmts.User")
       (effects (font (size 1 1) (thickness 0.15)))
     )
@@
     (pts (xy 160 140) (xy 160 110))
     (height 20)
-    (gr_text "30,0000 mm" (at 178.85 125 90) (layer "Cmts.User")
-      (effects (font (size 1 1) (thickness 0.15)))
-    )
+    (gr_text "1181,1024 mils" (at 178.85 125 90) (layer "Cmts.User")
+      (effects (font (size 1 1) (thickness 0.15)))
+    )
