File: HW/TestBoards/LNAs_EvalBoard/LNAs_EvalBoard.kicad_pcb (KiCad board)
At the start: 2 copper layers, 50 x 40 mm, 13 parts, among them J1 SMA, J2 SMA, J3 Picoblade_2x1_H, J4 Picoblade_2x1_H, U1 HMC342, U2 BFHK-2582+, U3 HMC342

Commit message: LO1 Eval Board
Parts:
- removed J4: Picoblade_2x1_H, Connector_Molex:Molex_PicoBlade_53261-0271_1x02-1MP_P1.25mm_Horizontal
- added H1: M2.5, MountingHole:MountingHole_2.7mm_M2.5_Pad, F.Cu at (124.0, 80.0)
- added H2: M2.5, MountingHole:MountingHole_2.7mm_M2.5_Pad, F.Cu at (124.0, 110.0)
- added H3: M2.5, MountingHole:MountingHole_2.7mm_M2.5_Pad, F.Cu at (164.0, 80.0)
- added H4: M2.5, MountingHole:MountingHole_2.7mm_M2.5_Pad, F.Cu at (164.0, 110.0)
- J3: value Picoblade_2x1_H -> Conn_01x04; footprint Connector_Molex:Molex_PicoBlade_53261-0271_1x02-1MP_P1.25mm_Horizontal -> Connector_PinSocket_2.00mm:PinSocket_1x04_P2.00mm_Vertical
- moved J3 8.51 mm to (142.0, 79.0), turned to 90 degrees
Routing:
- net VDD: track 24.8 -> 41.8 mm
- net GND: vias 198 -> 190
Other:
- board text added: "GND"
- board text added: "Vdd1"
- board text added: "Vdd2"

Commit message: All Test Boards developed
Routing:
- net GND: vias 190 -> 249

Commit message: Added Evaluation Boards for RO4003C 1.52 mm
Parts:
- J1, J2: footprint GGS_Connectors:LINX_CONSMA020.062-G -> GGS_Connectors:Johnson_142-0761-861
- moved J1 10.8 mm to (130.4, 95.0), turned to 90 degrees
- moved J2 10.6 mm to (157.8, 95.0), turned to -90 degrees
- moved J3 4.00 mm to (142.0, 83.0)
Connections:
- J3 pad 3: VDD -> GND
- J3 pad 4: GND -> VDD
Routing:
- net GND: track 0.95 -> 17.0 mm
- net VDD: track 41.8 -> 32.7 mm
- net /RF_Out: track 9.54 -> 11.7 mm
- net /RF_In: track 9.56 -> 10.9 mm
