File: HW/TestBoards/LNAs_EvalBoard/LNAs_EvalBoard_Ro4003C_60mils.kicad_pcb (KiCad board)
At the start: 2 copper layers, 50 x 40 mm, 12 parts, among them J1 SMA, J2 SMA, J3 Conn_01x04, U1 HMC342, U2 BFHK-2582+, U3 HMC342

Commit message: IDK
Parts:
- J3: footprint Connector_PinSocket_2.00mm:PinSocket_1x04_P2.00mm_Vertical -> Connector_PinHeader_2.54mm:PinHeader_1x04_P2.54mm_Vertical
Routing:
- net VDD: track 32.7 -> 31.0 mm
Changed lines of the file:
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@@
     )
   )
-  (footprint "Connector_PinSocket_2.00mm:PinSocket_1x04_P2.00mm_Vertical" (layer "F.Cu")
+  (footprint "Connector_PinHeader_2.54mm:PinHeader_1x04_P2.54mm_Vertical" (layer "F.Cu")
     (at 142 83 90)
-    (descr "Through hole straight socket strip, 1x04, 2.00mm pitch, single row (from Kicad 4.0.7), script generated")
-    (tags "Through hole socket strip THT 1x04 2.00mm single row")
+    (descr "Through hole straight pin header, 1x04, 2.54mm pitch, single row")
+    (tags "Through hole pin header THT 1x04 2.54mm single row")
     (property "Sheetfile" "LNAs_EvalBoard.kicad_sch")
     (property "Sheetname" "")
     (attr through_hole)
-    (fp_text reference "J3" (at 0 9 180) (layer "F.SilkS")
-      (effects (font (size 1 1) (thickness 0.15)))
-    )
-    (fp_text value "Conn_01x04" (at 0 8.5 90) (layer "F.Fab")
-      (effects (font (size 1 1) (thickness 0.15)))
-    )
-    (fp_text user "${REFERENCE}" (at 0 3) (layer "F.Fab")
-      (effects (font (size 1 1) (thickness 0.15)))
-    )
-    (fp_line (start -1.06 1) (end -1.06 7.06) (layer "F.SilkS") (width 0.12))
-    (fp_line (start 0 -1.06) (end 1.06 -1.06) (layer "F.SilkS") (width 0.12))
-    (fp_line (start 1.06 1) (end 1.06 7.06) (layer "F.SilkS") (width 0.12))
-    (fp_line (start 1.06 -1.06) (end 1.06 0) (layer "F.SilkS") (width 0.12))
-    (fp_line (start -1.06 1) (end 1.06 1) (layer "F.SilkS") (width 0.12))
-    (fp_line (start -1.06 7.06) (end 1.06 7.06) (layer "F.SilkS") (width 0.12))
-    (fp_line (start 1.5 7.5) (end -1.5 7.5) (layer "F.CrtYd") (width 0.05))
-    (fp_line (start -1.5 7.5) (end -1.5 -1.5) (layer "F.CrtYd") (width 0.05))
-    (fp_line (start 1.5 -1.5) (end 1.5 7.5) (layer "F.CrtYd") (width 0.05))
-    (fp_line (start -1.5 -1.5) (end 1.5 -1.5) (layer "F.CrtYd") (width 0.05))
-    (fp_line (start 1 -0.5) (end 1 7) (layer "F.Fab") (width 0.1))
-    (fp_line (start 1 7) (end -1 7) (layer "F.Fab") (width 0.1))
-    (fp_line (start 0.5 -1) (end 1 -0.5) (layer "F.Fab") (width 0.1))
-    (fp_line (start -1 -1) (end 0.5 -1) (layer "F.Fab") (width 0.1))
-    (fp_line (start -1 7) (end -1 -1) (layer "F.Fab") (width 0.1))
-    (pad "1" thru_hole rect (at 0 0 90) (size 1.35 1.35) (drill 0.8) (layers *.Cu *.Mask)
+    (fp_text reference "J3" (at 0 -2.33 90) (layer "F.SilkS")
+      (effects (font (size 1 1) (thickness 0.15)))
+    )
+    (fp_text value "Conn_01x04" (at 0 9.95 90) (layer "F.Fab")
+      (effects (font (size 1 1) (thickness 0.15)))
+    )
+    (fp_text user "${REFERENCE}" (at 0 3.81 180) (layer "F.Fab")
+      (effects (font (size 1 1) (thickness 0.15)))
+    )
+    (fp_line (start 1.33 1.27) (end 1.33 8.95) (layer "F.SilkS") (width 0.12))
+    (fp_line (start -1.33 0) (end -1.33 -1.33) (layer "F.SilkS") (width 0.12))
+    (fp_line (start -1.33 1.27) (end -1.33 8.95) (layer "F.SilkS") (width 0.12))
+    (fp_line (start -1.33 1.27) (end 1.33 1.27) (layer "F.SilkS") (width 0.12))
+    (fp_line (start -1.33 8.95) (end 1.33 8.95) (layer "F.SilkS") (width 0.12))
+    (fp_line (start -1.33 -1.33) (end 0 -1.33) (layer "F.SilkS") (width 0.12))
+    (fp_line (start -1.8 9.4) (end 1.8 9.4) (layer "F.CrtYd") (width 0.05))
+    (fp_line (start 1.8 9.4) (end 1.8 -1.8) (layer "F.CrtYd") (width 0.05))
+    (fp_line (start 1.8 -1.8) (end -1.8 -1.8) (layer "F.CrtYd") (width 0.05))
+    (fp_line (start -1.8 -1.8) (end -1.8 9.4) (layer "F.CrtYd") (width 0.05))
+    (fp_line (start 1.27 8.89) (end -1.27 8.89) (layer "F.Fab") (width 0.1))
+    (fp_line (start -1.27 -0.635) (end -0.635 -1.27) (layer "F.Fab") (width 0.1))
+    (fp_line (start -1.27 8.89) (end -1.27 -0.635) (layer "F.Fab") (width 0.1))
+    (fp_line (start 1.27 -1.27) (end 1.27 8.89) (layer "F.Fab") (width 0.1))
+    (fp_line (start -0.635 -1.27) (end 1.27 -1.27) (layer "F.Fab") (width 0.1))
+    (pad "1" thru_hole rect (at 0 0 90) (size 1.7 1.7) (drill 1) (layers *.Cu *.Mask)
       (net 1 "VDD") (pinfunction "Pin_1") (pintype "passive"))
-    (pad "2" thru_hole oval (at 0 2 90) (size 1.35 1.35) (drill 0.8) (layers *.Cu *.Mask)
+    (pad "2" thru_hole oval (at 0 2.54 90) (size 1.7 1.7) (drill 1) (layers *.Cu *.Mask)
       (net 2 "GND") (pinfunction "Pin_2") (pintype "passive"))
-    (pad "3" thru_hole oval (at 0 4 90) (size 1.35 1.35) (drill 0.8) (layers *.Cu *.Mask)
+    (pad "3" thru_hole oval (at 0 5.08 90) (size 1.7 1.7) (drill 1) (layers *.Cu *.Mask)
       (net 2 "GND") (pinfunction "Pin_3") (pintype "passive"))
-    (pad "4" thru_hole oval (at 0 6 90) (size 1.35 1.35) (drill 0.8) (layers *.Cu *.Mask)
+    (pad "4" thru_hole oval (at 0 7.62 90) (size 1.7 1.7) (drill 1) (layers *.Cu *.Mask)
       (net 1 "VDD") (pinfunction "Pin_4") (pintype "passive"))
-    (model "${KICAD6_3DMODEL_DIR}/Connector_PinSocket_2.00mm.3dshapes/PinSocket_1x04_P2.00mm_Vertical.wrl"
+    (model "${KICAD6_3DMODEL_DIR}/Connector_PinHeader_2.54mm.3dshapes/PinHeader_1x04_P2.54mm_Vertical.wrl"
       (offset (xyz 0 0 0))
       (scale (xyz 1 1 1))
@@
   )
   (segment (start 136.5 83) (end 134.098751 85.401249) (width 0.381) (layer "F.Cu") (net 1))
-  (segment (start 136.5 83) (end 142 83) (width 0.381) (layer "F.Cu") (net 1))
-  (segment (start 153 83) (end 148 83) (width 0.381) (layer "F.Cu") (net 1))
-  (segment (start 134.098751 85.401249) (end 134.098751 93.262499) (width 0.381) (layer "F.Cu") (net 1))
   (segment (start 154.401238 84.401238) (end 153 83) (width 0.381) (layer "F.Cu") (net 1))
   (segment (start 154.401238 93.312499) (end 154.401238 84.401238) (width 0.381) (layer "F.Cu") (net 1))
+  (segment (start 136.5 83) (end 142 83) (width 0.381) (layer "F.Cu") (net 1))
+  (segment (start 134.098751 85.401249) (end 134.098751 93.262499) (width 0.381) (layer "F.Cu") (net 1))
+  (segment (start 153 83) (end 149.62 83) (width 0.381) (layer "F.Cu") (net 1))
   (segment (start 143.944999 95) (end 143.95 95.005001) (width 0.381) (layer "F.Cu") (net 2))
   (segment (start 140 96.75) (end 148 96.75) (width 0.84074) (layer "F.Cu") (net 2))
