File: HW/TestBoards/IF2_EvalBoard/Mixer_2_RO4003C_60mils.kicad_pcb (KiCad board)
At the start: 2 copper layers, 60 x 30 mm, 19 parts, among them IC1 SIM-14+, IC2 LEE2-6+, IC3 LEE2-6+, J1 Conn_01x04, J2 SMA, J3 SMA, J4 SMA, J5 MS-156C3_20_, U1 B39871B4316P810

Commit message: IDK
Parts:
- J1: footprint Connector_PinHeader_1.27mm:PinHeader_1x04_P1.27mm_Vertical -> Connector_PinHeader_2.54mm:PinHeader_1x04_P2.54mm_Vertical
- moved J1 2.34 mm to (157.2, 98.7)
Routing:
- net /Vdd_amp1: track 9.16 -> 6.17 mm
- net /Vdd_amp2: track 9.07 -> 7.20 mm
- net /MS_out: track 0.09 -> 0.78 mm
- net GND: vias 0 -> 208
