File: HW/RFI-5G/RFI-5G_Interface/Boost1.kicad_sch (KiCad schematic)
At the start: 18 parts, among them U1 LT3048IDC-TRMPBF, U2 LT3048IDC-TRMPBF

Commit message: RF top and Bottom boards
Parts:
- L1, L2: value (none) -> 5.6 uH; footprint (none) -> ASPI4030S5R6M-T:ASPI-4030S-100M-T
Connections:
- net VCC renamed P/L power
Changed lines of the file:
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@@
+    )
+  )
+  (global_label "P{slash}L power" (shape input) (at 38.1 35.56 90) (fields_autoplaced)
+    (effects (font (size 1.27 1.27)) (justify left))
+    (property "Intersheet References" "${INTERSHEET_REFS}" (id 0) (at 38.0206 23.0474 90)
+      (effects (font (size 1.27 1.27)) (justify left) hide)
     )
   )
@@
     (effects (font (size 1.27 1.27)) (justify left))
     (property "Intersheet References" "${INTERSHEET_REFS}" (id 0) (at 206.7621 44.3706 0)
+      (effects (font (size 1.27 1.27)) (justify left) hide)
+    )
+  )
+  (global_label "P{slash}L power" (shape output) (at 36.83 111.76 90) (fields_autoplaced)
+    (effects (font (size 1.27 1.27)) (justify left))
+    (property "Intersheet References" "${INTERSHEET_REFS}" (id 0) (at 36.7506 99.2474 90)
       (effects (font (size 1.27 1.27)) (justify left) hide)
     )
@@
     (pin "1")
   )
-  (symbol (lib_id "power:VCC") (at 36.83 111.76 0) (unit 1)
-    (in_bom yes) (on_board yes) (fields_autoplaced)
-    (property "Reference" "#PWR0105" (id 0) (at 36.83 115.57 0)
-      (effects (font (size 1.27 1.27)) hide)
-    )
-    (property "Value" "VCC" (id 1) (at 36.83 106.68 0))
-    (property "Footprint" "" (id 2) (at 36.83 111.76 0)
-      (effects (font (size 1.27 1.27)) hide)
-    )
-    (property "Datasheet" "" (id 3) (at 36.83 111.76 0)
-      (effects (font (size 1.27 1.27)) hide)
-    )
-    (pin "1")
-  )
   (symbol (lib_id "Device:C") (at 76.2 127 0) (unit 1)
     (in_bom yes) (on_board yes) (fields_autoplaced)
@@
     (pin "1")
     (pin "2")
-  )
-  (symbol (lib_id "power:VCC") (at 38.1 35.56 0) (unit 1)
-    (in_bom yes) (on_board yes) (fields_autoplaced)
-    (property "Reference" "#PWR0103" (id 0) (at 38.1 39.37 0)
-      (effects (font (size 1.27 1.27)) hide)
-    )
-    (property "Value" "VCC" (id 1) (at 38.1 30.48 0))
-    (property "Footprint" "" (id 2) (at 38.1 35.56 0)
-      (effects (font (size 1.27 1.27)) hide)
-    )
-    (property "Datasheet" "" (id 3) (at 38.1 35.56 0)
-      (effects (font (size 1.27 1.27)) hide)
-    )
-    (pin "1")
   )
   (symbol (lib_id "Device:C") (at 176.53 59.69 0) (unit 1)
@@
     (in_bom yes) (on_board yes) (fields_autoplaced)
     (property "Reference" "L2" (id 0) (at 71.12 106.68 90))
-    (property "Value" "" (id 1) (at 71.12 109.22 90))
-    (property "Footprint" "" (id 2) (at 71.12 113.03 0)
+    (property "Value" "5.6 uH" (id 1) (at 71.12 109.22 90))
+    (property "Footprint" "ASPI4030S5R6M-T:ASPI-4030S-100M-T" (id 2) (at 71.12 113.03 0)
       (effects (font (size 1.27 1.27)) hide)
     )
@@
     (in_bom yes) (on_board yes) (fields_autoplaced)
     (property "Reference" "L1" (id 0) (at 72.39 30.48 90))
-    (property "Value" "" (id 1) (at 72.39 33.02 90))
-    (property "Footprint" "" (id 2) (at 72.39 36.83 0)
-      (effects (font (size 1.27 1.27)) hide)
-    )
+    (property "Value" "5.6 uH" (id 1) (at 72.39 33.02 90))
+    (property "Footprint" "ASPI4030S5R6M-T:ASPI-4030S-100M-T" (id 2) (at 72.39 36.83 0)
+      (effects (font (size 1.27 1.27)) hide)
+    )
