File: HW/RFI-5G/RFI-5G_Interface/Boost2.kicad_sch (KiCad schematic)
At the start: 9 parts, among them U3 LT3048IDC-TRMPBF

Commit message: RF top and Bottom boards
Parts:
- L3: value (none) -> 5.6 uH; footprint (none) -> ASPI4030S5R6M-T:ASPI-4030S-100M-T
Connections:
- net VCC renamed P/L power
Changed lines of the file:
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@@
     (stroke (width 0) (type default) (color 0 0 0 0))
+  )
+  (global_label "P{slash}L power" (shape output) (at 40.64 46.99 90) (fields_autoplaced)
+    (effects (font (size 1.27 1.27)) (justify left))
+    (property "Intersheet References" "${INTERSHEET_REFS}" (id 0) (at 40.5606 34.4774 90)
+      (effects (font (size 1.27 1.27)) (justify left) hide)
+    )
   )
   (global_label "13V" (shape output) (at 198.12 55.88 0) (fields_autoplaced)
@@
     )
     (property "Datasheet" "" (id 3) (at 46.99 63.5 0)
-      (effects (font (size 1.27 1.27)) hide)
-    )
-    (pin "1")
-  )
-  (symbol (lib_id "power:VCC") (at 40.64 46.99 0) (unit 1)
-    (in_bom yes) (on_board yes) (fields_autoplaced)
-    (property "Reference" "#PWR0107" (id 0) (at 40.64 50.8 0)
-      (effects (font (size 1.27 1.27)) hide)
-    )
-    (property "Value" "VCC" (id 1) (at 40.64 41.91 0))
-    (property "Footprint" "" (id 2) (at 40.64 46.99 0)
-      (effects (font (size 1.27 1.27)) hide)
-    )
-    (property "Datasheet" "" (id 3) (at 40.64 46.99 0)
       (effects (font (size 1.27 1.27)) hide)
     )
@@
     (in_bom yes) (on_board yes) (fields_autoplaced)
     (property "Reference" "L3" (id 0) (at 74.93 41.91 90))
-    (property "Value" "" (id 1) (at 74.93 44.45 90))
-    (property "Footprint" "" (id 2) (at 74.93 48.26 0)
+    (property "Value" "5.6 uH" (id 1) (at 74.93 44.45 90))
+    (property "Footprint" "ASPI4030S5R6M-T:ASPI-4030S-100M-T" (id 2) (at 74.93 48.26 0)
       (effects (font (size 1.27 1.27)) hide)
     )
