File: HW/RFI-5G/RFI-5G_Interface/LDOs.kicad_sch (KiCad schematic)
At the start: 20 parts, among them U4 MIC2215-AAAYML-TR, U5 MIC2215-AAAYML-TR

Commit message: RF top and Bottom boards
Parts:
- added C30, C32: 1 uF, Capacitor_SMD:C_0603_1608Metric_Pad1.08x0.95mm_HandSolder, symbol Device:C
- added C31, C33: 4.7 uF, Capacitor_SMD:C_0603_1608Metric_Pad1.08x0.95mm_HandSolder, symbol Device:C
- added R24, R25, R26, R27: X, Resistor_SMD:R_0603_1608Metric_Pad0.98x0.95mm_HandSolder, symbol Device:R
Connections:
- net VCC is gone; now on net P/L power: C13.1, C18.1, C28.1, C29.1, U4.12 (VIN3), U4.2 (VIN1), U4.3 (VIN2), U4.6 (EN1), U4.7 (EN2), U4.8 (EN3), U5.2 (VIN1), U5.6 (EN1)
- net GND: now also C30.2, C31.2, C32.2, C33.2, R25.1, R27.1
- net P/L power: now reaches U5.12 (VIN3)
- net P/L power: now also U5.3 (VIN2), U5.7 (EN2), U5.8 (EN3), C30.1, C32.1
- net LDO_extra2: now reaches U5.13 (VOUT3)
- net LDO_extra2: now also C33.1, R26.1
- net at U5.14 (ADJ3): now also R26.2, R27.2
- net LDO_extra1: now reaches U5.4 (VOUT2)
- net LDO_extra1: now also C31.1, R24.2
- net at U5.5 (ADJ2): now also R24.1, R25.2
- no-connect marks 8 -> 0
Other:
- moved on the sheet: C18
