File: HW/RFI-5G/RFI-5G_Interface/Vtune1.kicad_sch (KiCad schematic)
At the start: 4 parts

Commit message: RF top and Bottom boards
Connections:
- net VCC renamed P/L power
Changed lines of the file:
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@@
+    )
+  )
+  (global_label "P{slash}L power" (shape output) (at 72.39 36.83 90) (fields_autoplaced)
+    (effects (font (size 1.27 1.27)) (justify left))
+    (property "Intersheet References" "${INTERSHEET_REFS}" (id 0) (at 72.3106 24.3174 90)
+      (effects (font (size 1.27 1.27)) (justify left) hide)
     )
   )
@@
     (pin "2")
   )
-  (symbol (lib_id "power:VCC") (at 72.39 36.83 0) (unit 1)
-    (in_bom yes) (on_board yes) (fields_autoplaced)
-    (property "Reference" "#PWR0133" (id 0) (at 72.39 40.64 0)
-      (effects (font (size 1.27 1.27)) hide)
-    )
-    (property "Value" "VCC" (id 1) (at 72.39 31.75 0))
-    (property "Footprint" "" (id 2) (at 72.39 36.83 0)
-      (effects (font (size 1.27 1.27)) hide)
-    )
-    (property "Datasheet" "" (id 3) (at 72.39 36.83 0)
-      (effects (font (size 1.27 1.27)) hide)
-    )
-    (pin "1")
-  )
   (symbol (lib_id "power:GND") (at 91.44 59.69 0) (unit 1)
