File: HW/RFI-5G/RFI-5G_Interface/low_freq_board.kicad_pcb (KiCad board)
At the start: 4 copper layers, 40 x 40 mm, 70 parts, among them J1 Conn_01x10_Female, J2 Conn_01x10_Female, J3 Conn_01x10_Female, J4 Conn_01x10_Female, J5 Conn_01x04_Female, U1 LT3048IDC-TRMPBF, U2 LT3048IDC-TRMPBF, U3 LT3048IDC-TRMPBF, U4 MIC2215-AAAYML-TR, U5 MIC2215-AAAYML-TR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

Commit message: RF top and Bottom boards
Parts:
- added C30: 1 uF, Capacitor_SMD:C_0603_1608Metric_Pad1.08x0.95mm_HandSolder, B.Cu at (103.5, 74.7)
- added C31: 4.7 uF, Capacitor_SMD:C_0603_1608Metric_Pad1.08x0.95mm_HandSolder, B.Cu at (99.5, 82.5)
- added C32: 1 uF, Capacitor_SMD:C_0603_1608Metric_Pad1.08x0.95mm_HandSolder, B.Cu at (103.3, 82.5)
- added C33: 4.7 uF, Capacitor_SMD:C_0603_1608Metric_Pad1.08x0.95mm_HandSolder, B.Cu at (103.9, 73.1)
- added R24: X, Resistor_SMD:R_0603_1608Metric_Pad0.98x0.95mm_HandSolder, B.Cu at (99.5, 79.1)
- added R25: X, Resistor_SMD:R_0603_1608Metric_Pad0.98x0.95mm_HandSolder, B.Cu at (99.5, 75.8)
- added R26: X, Resistor_SMD:R_0603_1608Metric_Pad0.98x0.95mm_HandSolder, B.Cu at (106.4, 76.4)
- added R27: X, Resistor_SMD:R_0603_1608Metric_Pad0.98x0.95mm_HandSolder, B.Cu at (107.4, 73.9)
- J1, J4: value Conn_01x10_Female -> Conn_01x03; footprint easyeda:CES-110-XX-Y-S -> Connector_PinHeader_2.54mm:PinHeader_1x03_P2.54mm_Vertical
- J2: value Conn_01x10_Female -> Conn_01x02; footprint easyeda:CES-110-XX-Y-S -> Connector_PinHeader_2.54mm:PinHeader_1x02_P2.54mm_Vertical
- J3: value Conn_01x10_Female -> Conn_01x10; footprint easyeda:CES-110-XX-Y-S -> Connector_PinHeader_2.54mm:PinHeader_1x10_P2.54mm_Vertical
- J5: value Conn_01x04_Female -> Conn_01x06_Female; footprint Connector_PinHeader_2.54mm:PinHeader_1x04_P2.54mm_Vertical -> Connector_PinHeader_1.00mm:PinHeader_1x06_P1.00mm_Vertical
- L1, L2, L3: footprint footprints:ASPI-4030S-5R6M-T -> ASPI4030S5R6M-T:ASPI-4030S-100M-T
- moved R8 56.3 mm to (115.0, 82.4), turned to 90 degrees
- moved R12 54.2 mm to (115.0, 72.4), turned to -90 degrees
- moved R7 54.0 mm to (115.0, 79.1), turned to -90 degrees
- moved C15 54.0 mm to (112.7, 82.4), turned to -90 degrees
- moved R11 52.9 mm to (115.0, 75.7), turned to 90 degrees
- moved C16 51.7 mm to (113.5, 73.0), turned to 90 degrees
- moved C13 49.9 mm to (111.2, 82.4), turned to -90 degrees
- moved C29 46.8 mm to (112.0, 73.0), turned to 90 degrees
- moved C28 46.8 mm to (109.7, 81.7), turned to -90 degrees
- moved U4 46.5 mm to (111.6, 77.4), turned to 90 degrees
- moved C17 44.5 mm to (108.1, 83.1), turned to -90 degrees
- moved C14 42.2 mm to (110.2, 73.6), turned to 90 degrees
- moved R9 41.1 mm to (108.1, 79.7), turned to 90 degrees
- moved U2 40.6 mm to (111.2, 65.8)
- moved C7 40.6 mm to (110.8, 68.5)
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Connections:
- C1 pad 1: VCC -> P/L power
- C13 pad 1: VCC -> P/L power
- C18 pad 1: VCC -> P/L power
- C24 pad 1: VCC -> P/L power
- C25 pad 1: VCC -> P/L power
- C27 pad 1: VCC -> P/L power
- C28 pad 1: VCC -> P/L power
- C29 pad 1: VCC -> P/L power
- C5 pad 1: VCC -> P/L power
- C9 pad 1: VCC -> P/L power
- J1 pad 3: RX -> GND
- J2 pad 1: L2BURN -> GND
- J2 pad 2: PALE -> VCC
- J3 pad 1: CHRG -> 2V75
- J3 pad 10: OLAR_Z -> GND
- J3 pad 2: FAULT -> Vtune2
- J3 pad 3: 3 -> GND
- J3 pad 4: unconnected-(J3-Pad4) -> GND
- J3 pad 5: unconnected-(J3-Pad5) -> P/L power
- J3 pad 6: unconnected-(J3-Pad6) -> LEE1_Vcc
- J3 pad 7: unconnected-(J3-Pad7) -> LEE2_Vcc
- J3 pad 8: MPPT_Y -> 3V
- J3 pad 9: MPPT_Z -> RSSI
- J4 pad 1: PCLK -> GND
- J5 pad 1: unconnected-(J5-Pad1) -> Vtune1
- J5 pad 2: unconnected-(J5-Pad2) -> 2V5
- J5 pad 3: unconnected-(J5-Pad3) -> LDO_extra1
- J5 pad 4: unconnected-(J5-Pad4) -> 2V7
- L1 pad 1: VCC -> P/L power
- L2 pad 1: VCC -> P/L power
- L3 pad 1: VCC -> P/L power
- R17 pad 1: VCC -> P/L power
- R20 pad 1: VCC -> P/L power
- R21 pad 1: VCC -> P/L power
- U1 pad 2: VCC -> P/L power
- U1 pad 7: VCC -> P/L power
- U2 pad 2: VCC -> P/L power
- U2 pad 7: VCC -> P/L power
- U3 pad 2: VCC -> P/L power
- U3 pad 7: VCC -> P/L power
- U4 pad 12: VCC -> P/L power
- U4 pad 2: VCC -> P/L power
- U4 pad 3: VCC -> P/L power
- U4 pad 6: VCC -> P/L power
- U4 pad 7: VCC -> P/L power
- U4 pad 8: VCC -> P/L power
- U5 pad 12: unconnected-(U5-Pad12) -> P/L power
- U5 pad 13: unconnected-(U5-Pad13) -> LDO_extra2
- U5 pad 14: unconnected-(U5-Pad14) -> Net-(R26-Pad2)
- U5 pad 2: VCC -> P/L power
- U5 pad 3: unconnected-(U5-Pad3) -> P/L power
- U5 pad 4: unconnected-(U5-Pad4) -> LDO_extra1
- U5 pad 5: unconnected-(U5-Pad5) -> Net-(R24-Pad1)
- U5 pad 6: VCC -> P/L power
- U5 pad 7: unconnected-(U5-Pad7) -> P/L power
- U5 pad 8: unconnected-(U5-Pad8) -> P/L power
Routing:
- net P/L power: track 0.00 -> 44.8 mm, vias 0 -> 26
- net LEE1_Vcc: track 3.98 -> 47.8 mm
- net 2V75: track 3.94 -> 46.9 mm, vias 0 -> 1
- net VCC: track 34.2 -> 0.00 mm, vias 24 -> 0
- net RSSI: track 0.71 -> 31.3 mm
- net LEE2_Vcc: track 3.97 -> 33.2 mm
- net LDO_extra1: track 0.00 -> 21.4 mm, vias 0 -> 1
- net 2V5: track 5.39 -> 17.2 mm, vias 0 -> 1
- net 2V7: track 4.67 -> 15.9 mm, vias 0 -> 1
- net 3V: track 5.41 -> 15.6 mm, vias 0 -> 1
- net LDO_extra2: track 0.00 -> 10.00 mm
- net GND: track 66.7 -> 58.2 mm, vias 52 -> 144
- net Vtune2: track 1.22 -> 8.72 mm
- net Vtune1: track 4.98 -> 11.9 mm, vias 1 -> 0
- net Net-(R26-Pad2): track 0.00 -> 5.75 mm
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- added copper zone on B.Cu, net P/L power
- added copper zone on In1.Cu, net P/L power
- removed copper zone on B.Cu, net VCC
- removed copper zone on In1.Cu, net VCC
Other:
- board text added: "( .ω.)"
- board text added: "Nanosatlab, ETSETB, UPC"
- board text added: "ʕっ•ᴥ•ʔっ"

Commit message: PL boards
Parts:
- J5: value Conn_01x06_Female -> Conn_01x10_Female; footprint Connector_PinHeader_1.00mm:PinHeader_1x06_P1.00mm_Vertical -> Connector_PinHeader_1.00mm:PinHeader_1x10_P1.00mm_Vertical; moved to F.Cu
- moved J5 2.00 mm to (99.4, 70.3), turned to 90 degrees
Connections:
- J5 pad 1: Vtune1 -> Vcc_IF1Amp
- J5 pad 2: 2V5 -> VTune1
- J5 pad 3: LDO_extra1 -> Vcc_VCO
- J5 pad 4: 2V7 -> Vcc_LO1Amp
- J5 pad 5: LDO_extra2 -> Vcc_LNA2
- J5 pad 6: 2V75 -> Vcc_LNA1

Commit message: idk
Routing:
- net GND: vias 144 -> 139
Changed lines of the file:
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@@
       (rotate (xyz 0 0 0))
     )
+    (model "C:/Users/guill/Documents/GitHub/NSL_KiCad_Libraries/Power/StepFiles/MLF16_4X4_MCH.step"
+      (offset (xyz 0 0 0))
+      (scale (xyz 1 1 1))
+      (rotate (xyz 0 0 0))
+    )
   )
   (footprint "Capacitor_SMD:C_0603_1608Metric_Pad1.08x0.95mm_HandSolder" (layer "B.Cu")
@@
       (rotate (xyz 0 0 0))
     )
+    (model "C:/Users/guill/Documents/GitHub/NSL_KiCad_Libraries/Power/StepFiles/MLF16_4X4_MCH.step"
+      (offset (xyz 0 0 0))
+      (scale (xyz 1 1 1))
+      (rotate (xyz 0 0 0))
+    )
   )
   (footprint "Capacitor_SMD:C_0603_1608Metric_Pad1.08x0.95mm_HandSolder" (layer "B.Cu")
@@
       (rotate (xyz -90 0 90))
     )
+    (model "C:/Users/guill/Documents/GitHub/NSL_KiCad_Libraries/Miscellaneous/StepFiles/Abracon_ASPI-4030S-5R6M-T.step"
+      (offset (xyz 0 0 0))
+      (scale (xyz 1 1 1))
+      (rotate (xyz 0 0 0))
+    )
   )
   (footprint "Resistor_SMD:R_0603_1608Metric_Pad0.98x0.95mm_HandSolder" (layer "B.Cu")
@@
     (pad "2" smd rect locked (at 1.3462 0 90) (size 3.5052 1.8034) (layers "B.Cu" "B.Paste" "B.Mask")
       (net 25 "Net-(L2-Pad2)") (pinfunction "2") (pintype "passive"))
-    (model "C:/Users/maarc/Downloads/ASPI-4030S-5R6M-T--3DModel-STEP-400430.STEP"
+    (model "C:/Users/maarc/Downloads/ASPI-4030S-5R6M-T--3DModel-STEP-400430.STEP" hide
       (offset (xyz 0 0 0))
       (scale (xyz 1 1 1))
       (rotate (xyz -90 0 90))
     )
+    (model "C:/Users/guill/Documents/GitHub/NSL_KiCad_Libraries/Miscellaneous/StepFiles/Abracon_ASPI-4030S-5R6M-T.step"
+      (offset (xyz 0 0 0))
+      (scale (xyz 1 1 1))
+      (rotate (xyz 0 0 0))
+    )
   )
   (footprint "Capacitor_SMD:C_0603_1608Metric_Pad1.08x0.95mm_HandSolder" (layer "B.Cu")
@@
       (rotate (xyz 0 0 0))
     )
+    (model "C:/Users/guill/Documents/GitHub/NSL_KiCad_Libraries/Power/StepFiles/MLF16_4X4_MCH.step"
+      (offset (xyz 0 0 0))
+      (scale (xyz 1 1 1))
+      (rotate (xyz 0 0 0))
+    )
   )
   (footprint "Resistor_SMD:R_0603_1608Metric_Pad0.98x0.95mm_HandSolder" (layer "B.Cu")
@@
     (pad "2" smd rect locked (at 1.3462 0 90) (size 3.5052 1.8034) (layers "B.Cu" "B.Paste" "B.Mask")
       (net 24 "Net-(L1-Pad2)") (pinfunction "2") (pintype "passive"))
-    (model "C:/Users/maarc/Downloads/ASPI-4030S-5R6M-T--3DModel-STEP-400430.STEP"
+    (model "C:/Users/maarc/Downloads/ASPI-4030S-5R6M-T--3DModel-STEP-400430.STEP" hide
       (offset (xyz 0 0 0))
       (scale (xyz 1 1 1))
       (rotate (xyz -90 0 90))
     )
+    (model "C:/Users/guill/Documents/GitHub/NSL_KiCad_Libraries/Miscellaneous/StepFiles/Abracon_ASPI-4030S-5R6M-T.step"
+      (offset (xyz 0 0 0))
+      (scale (xyz 1 1 1))
+      (rotate (xyz 0 0 0))
+    )
   )
   (footprint "Resistor_SMD:R_0603_1608Metric_Pad0.98x0.95mm_HandSolder" (layer "B.Cu")
@@
   (via (at 100.569455 64.272193) (size 0.4) (drill 0.2) (layers "F.Cu" "B.Cu") (net 2))
   (via (at 88.872893 77.935278) (size 0.4) (drill 0.2) (layers "F.Cu" "B.Cu") (free) (net 2))
-  (via (at 99.212893 69.722893) (size 0.4) (drill 0.2) (layers "F.Cu" "B.Cu") (free) (net 2))
   (via (at 113.490393 71.250393) (size 0.4) (drill 0.2) (layers "F.Cu" "B.Cu") (net 2))
   (via (at 101.089554 86.081939) (size 0.4) (drill 0.2) (layers "F.Cu" "B.Cu") (free) (net 2))
@@
   (via (at 117.112893 81.902416) (size 0.4) (drill 0.2) (layers "F.Cu" "B.Cu") (free) (net 2))
   (via (at 97.130985 86.081939) (size 0.4) (drill 0.2) (layers "F.Cu" "B.Cu") (free) (net 2))
-  (via (at 99.952893 69.722893) (size 0.4) (drill 0.2) (layers "F.Cu" "B.Cu") (free) (net 2))
   (via (at 117.132893 64.710985) (size 0.4) (drill 0.2) (layers "F.Cu" "B.Cu") (free) (net 2))
   (via (at 112.961927 57.892893) (size 0.4) (drill 0.2) (layers "F.Cu" "B.Cu") (free) (net 2))
@@
   (via (at 109.006692 86.081939) (size 0.4) (drill 0.2) (layers "F.Cu" "B.Cu") (free) (net 2))
   (via (at 117.132893 63.391462) (size 0.4) (drill 0.2) (layers "F.Cu" "B.Cu") (free) (net 2))
-  (via (at 108.452893 69.832893) (size 0.4) (drill 0.2) (layers "F.Cu" "B.Cu") (free) (net 2))
   (via (at 114.582893 60.032893) (size 0.4) (drill 0.2) (layers "F.Cu" "B.Cu") (free) (net 2))
   (via (at 96.070393 76.855393) (size 0.4) (drill 0.2) (layers "F.Cu" "B.Cu") (net 2))
@@
   (via (at 92.088855 64.119181) (size 0.4) (drill 0.2) (layers "F.Cu" "B.Cu") (net 2))
   (via (at 110.940393 74.470393) (size 0.4) (drill 0.2) (layers "F.Cu" "B.Cu") (net 2))
-  (via (at 107.662893 69.832893) (size 0.4) (drill 0.2) (layers "F.Cu" "B.Cu") (free) (net 2))
   (via (at 88.872893 76.615755) (size 0.4) (drill 0.2) (layers "F.Cu" "B.Cu") (free) (net 2))
   (via (at 111.178343 65.800393) (size 0.4) (drill 0.2) (layers "F.Cu" "B.Cu") (net 2))
   (via (at 117.122893 79.258123) (size 0.4) (drill 0.2) (layers "F.Cu" "B.Cu") (free) (net 2))
-  (via (at 98.502893 69.722893) (size 0.4) (drill 0.2) (layers "F.Cu" "B.Cu") (free) (net 2))
   (via (at 94.491939 86.081939) (size 0.4) (drill 0.2) (layers "F.Cu" "B.Cu") (free) (net 2))
   (via (at 109.080393 64.160393) (size 0.4) (drill 0.2) (layers "F.Cu" "B.Cu") (net 2))
