File: HW/RFI-5G/RFI-5G_Interface/low_freq_board.kicad_sch (KiCad schematic)
At the start: 0 parts

Commit message: RF top and Bottom boards
Other:
- note added: "Vcc will need to be changed to PoL whena pin for the point of load is available. Also, in the PCB, the Vcc zone will have to be changed to PoL."
